Commit message: Fix gazebo robot description issue

File: go2_description/xacro/const.xacro (robot description, xacro)
@@ -71,10 +71,4 @@
     <xacro:property name="trunk_iyz" value="0"/>
     <xacro:property name="trunk_izz" value="0.055683"/>
-    <!-- <xacro:property name="trunk_ixx" value="0.02448"/>
-    <xacro:property name="trunk_ixy" value="0.00012166"/>
-    <xacro:property name="trunk_ixz" value="0.0014849"/>
-    <xacro:property name="trunk_iyy" value="0.098077"/>
-    <xacro:property name="trunk_iyz" value="-3.12E-05"/>
-    <xacro:property name="trunk_izz" value="0.107"/> -->
     <!-- hip (left front) -->
     <xacro:property name="hip_mass" value="0.678"/>

File: go2_description/xacro/go2_robot.xacro (robot description, xacro)
@@ -5,8 +5,4 @@
     <xacro:include filename="$(find go2_description)/xacro/materials.xacro"/>
     <xacro:include filename="$(find go2_description)/xacro/go2_leg.xacro"/>
-    <!-- <xacro:include filename="/home/e-yantra/unitree_ws/install/go2_description/share/go2_description/xacro/const.xacro"/>
-    <xacro:include filename="/home/e-yantra/unitree_ws/install/go2_description/share/go2_description/xacro/materials.xacro"/>
-    <xacro:include filename="/home/e-yantra/unitree_ws/install/go2_description/share/go2_description/xacro/leg.xacro"/> -->
-    <!-- <xacro:include filename="/home/e-yantra/unitree_ws/install/go2_description/share/go2_description/xacro/leg.xacro"/> -->
     <!-- find-pkg-share -->
     <!-- <xacro:include filename="$(find go2_description)/xacro/stairs.xacro"/> -->
@@ -16,14 +12,4 @@
     <!-- Rotor related joint and link is only for demonstrate location. -->
     <!-- Actually, the rotor will rotate and the joint is not fixed. Reduction ratio should be considered. -->
-    <!-- Debug mode will hung up the robot, use "true" or "false" to switch it. -->
-    <!-- <xacro:if value="$(arg DEBUG)">
-    </xacro:if>  -->
-    <!-- <link name="world"/>
-    <link name="map"/>
-    <joint name="base_static_joint" type="fixed">
-        <origin rpy="0 0 0" xyz="0 0 0"/>
-        <parent link="world"/>
-        <child link="map"/>
-    </joint> -->
     <xacro:include filename="$(find go2_description)/xacro/accessories.urdf.xacro" />
     <xacro:include filename="$(find go2_description)/xacro/camera.xacro" />
@@ -61,8 +47,4 @@
             <!-- <mass value="2"/> -->
             <mass value="${trunk_mass}"/>
-            <!-- <inertia
-                ixx="0.02448" ixy="0.00012166" ixz="0.0014849"
-                iyy="0.098077" iyz="-3.12E-05"
-                izz="0.107"/>   -->
             <inertia
                 ixx="${trunk_ixx}" ixy="${trunk_ixy}" ixz="${trunk_ixz}"
@@ -76,55 +58,4 @@
         base_height="0.114"
     />
-    <!-- <joint name="imu_joint" type="fixed">
-        <parent link="trunk"/>
-        <child link="imu_link"/>
-        <origin rpy="0 0 0" xyz="0 0 0"/>
-    </joint>
-    <link name="imu_link">
-        <inertial>
-            <mass value="0.001"/>
-            <origin rpy="0 0 0" xyz="0 0 0"/>
-            <inertia ixx="0.0001" ixy="0" ixz="0" iyy="0.0001" iyz="0" izz="0.0001"/>
-        </inertial>
-        <visual>
-            <origin rpy="0 0 0" xyz="0 0 0"/>
-            <geometry>
-                <box size="0.001 0.001 0.001"/>
-            </geometry>
-            <material name="red"/>
-        </visual>
-        <collision>
-            <origin rpy="0 0 0" xyz="0 0 0"/>
-            <geometry>
-                <box size=".001 .001 .001"/>
-            </geometry>
-        </collision>
-    </link> -->
-    <!--
-    <joint name="load_joint" type="fixed">
-        <parent link="trunk"/>
-        <child link="load_link"/>
-        <origin rpy="0 0 0" xyz="0 0 0"/>
-    </joint>
-    <link name="load_link">
-        <inertial>
-            <mass value="5"/>
-            <origin rpy="0 0 0" xyz="0 0 0"/>
-            <inertia ixx="0.01" ixy="0" ixz="0" iyy="0.01" iyz="0" izz="0.01"/>
-        </inertial>
-        <visual>
-            <origin rpy="0 0 0" xyz="0 0 0.2"/>
-            <geometry>
-                <box size="0.5 0.3 0.2"/>
-            </geometry>
-        </visual>
-        <collision>
-            <origin rpy="0 0 0" xyz="0 0 0"/>
-            <geometry>
-                <box size=".001 .001 .001"/>
-            </geometry>
-        </collision>
-    </link>
--->
     <xacro:leg name="lf" mirror="1"  mirror_dae="True"   front_hind="1"  front_hind_dae="True"  />
     <xacro:leg name="rf" mirror="-1" mirror_dae= "False" front_hind="1"  front_hind_dae="True"  />
@@ -147,6 +78,4 @@
         <plugin filename="libgazebo_ros2_control.so" name="gazebo_ros2_control">
             <parameters>$(find go2_description)/config/go2_ros_control.yaml</parameters>
-            <robot_param>robot_description</robot_param>
-            <robot_param_node>robot_state_publisher</robot_param_node>
         </plugin>
     </gazebo>
