Commit message: fix: collapse multiline XML comments to prevent gazebo_ros2_control parser error
Multiline XML comments in accessories.urdf.xacro, camera.xacro, and
hokuyo_utm30lx.urdf.xacro embedded literal newlines into the generated
URDF string. When gazebo_ros2_control receives robot_description as a
--param shell argument, those newlines break the parameter parser with
"Couldn't parse parameter override rule".

All multiline comments collapsed to single-line equivalents. No
functional change to the robot description.

Fixes #2

File: go2_description/xacro/accessories.urdf.xacro (robot description, xacro)
@@ -4,14 +4,5 @@
         <xacro:include filename="$(find go2_description)/xacro/hokuyo_utm30lx.urdf.xacro" />
         <!-- <xacro:include filename="$(find go2_description)/xacro/asus_camera.urdf.xacro" /> -->
-        <!-- <xacro:hokuyo_utm30lx
-            name="hokuyo"
-            parent="${base_name}"
-            ros_topic="scan"
-            update_rate="30"
-            ray_count="1040"
-            min_angle="130"
-            max_angle="-130" >
-            <origin xyz="0.0 0.0 ${base_height / 2 + 0.04}" rpy="0 0 0"/>
-        </xacro:hokuyo_utm30lx> -->
+        <!-- <xacro:hokuyo_utm30lx name="hokuyo" parent="${base_name}" ros_topic="scan" update_rate="30" ray_count="1040" min_angle="130" max_angle="-130"><origin xyz="0.0 0.0 ${base_height / 2 + 0.04}" rpy="0 0 0"/></xacro:hokuyo_utm30lx> -->
         <!-- hls_lfcd_lds -->
         <xacro:hokuyo_utm30lx
@@ -25,9 +16,5 @@
             <origin xyz="0.0 0.0 ${base_height / 2 + 0.04}" rpy="0 0 0"/>
         </xacro:hokuyo_utm30lx>
-        <!-- <xacro:asus_camera
-            parent="${base_name}"
-            name="camera">
-            <origin xyz="${base_length / 2} 0.0 -${base_height / 2 + 0.01}" rpy="0 0 0"/>
-        </xacro:asus_camera> -->
+        <!-- <xacro:asus_camera parent="${base_name}" name="camera"><origin xyz="${base_length / 2} 0.0 -${base_height / 2 + 0.01}" rpy="0 0 0"/></xacro:asus_camera> -->
         <link name="imu_link">
             <inertial>
@@ -51,24 +38,9 @@
                             <remapping>~/out:=data</remapping>
                         </ros>
-                        <!-- <updateRate>50.0</updateRate>
-                        <bodyName>imu_link</bodyName>
-                        <topicName>imu/data</topicName>
-                        <accelDrift>0.005 0.005 0.005</accelDrift>
-                        <accelGaussianNoise>0.005 0.005 0.005</accelGaussianNoise>
-                        <rateDrift>0.005 0.005 0.005 </rateDrift>
-                        <rateGaussianNoise>0.005 0.005 0.005 </rateGaussianNoise>
-                        <headingDrift>0.005</headingDrift>
-                        <headingGaussianNoise>0.005</headingGaussianNoise> -->
+                        <!-- <updateRate>50.0</updateRate><bodyName>imu_link</bodyName><topicName>imu/data</topicName><accelDrift>0.005 0.005 0.005</accelDrift><accelGaussianNoise>0.005 0.005 0.005</accelGaussianNoise><rateDrift>0.005 0.005 0.005</rateDrift><rateGaussianNoise>0.005 0.005 0.005</rateGaussianNoise><headingDrift>0.005</headingDrift><headingGaussianNoise>0.005</headingGaussianNoise> -->
                     </plugin>
                 </sensor>
             </gazebo>
-        <!-- <xacro:include filename="$(find velodyne_description)/urdf/VLP-16.urdf.xacro"/>
-        <xacro:VLP-16 parent="${base_name}" name="velodyne" topic="velodyne_points" hz="10" samples="1024" gpu="false" lasers="16" max_range="100">
-            <origin xyz="0 0 ${base_height / 2}" rpy="0 0 0" />
-        </xacro:VLP-16>
-        <xacro:include filename="$(find champ_arm_description)/urdf/champ_arm.urdf.xacro" />
-        <xacro:champ_arm parent="${base_name}">
-            <origin xyz="0.07 0.0 ${base_height / 2}" rpy="0 0 0"/>
-        </xacro:champ_arm> -->
+        <!-- <xacro:include filename="$(find velodyne_description)/urdf/VLP-16.urdf.xacro"/><xacro:VLP-16 parent="${base_name}" name="velodyne" topic="velodyne_points" hz="10" samples="1024" gpu="false" lasers="16" max_range="100"><origin xyz="0 0 ${base_height / 2}" rpy="0 0 0"/></xacro:VLP-16><xacro:include filename="$(find champ_arm_description)/urdf/champ_arm.urdf.xacro"/><xacro:champ_arm parent="${base_name}"><origin xyz="0.07 0.0 ${base_height / 2}" rpy="0 0 0"/></xacro:champ_arm> -->
     </xacro:macro>
 </robot>

File: go2_description/xacro/camera.xacro (robot description, xacro)
@@ -1,16 +1,7 @@
-<!-- GO2 Robot Description with RGB-D Camera Plugin
-     Based on: https://github.com/arjun-sadananda/go2_nav2_ros2
-     Added: Gazebo RGB-D camera plugin for YOLOv8 + depth
-     Full mesh files and full URDF come from the upstream go2_nav2_ros2 repo.
-     Clone it and use go2_description from there — this file shows
-     the camera xacro addition to include in go2_robot.xacro.
--->
+<!-- GO2 Robot Description with RGB-D Camera Plugin. Based on: https://github.com/arjun-sadananda/go2_nav2_ros2. Added: Gazebo RGB-D camera plugin for YOLOv8 + depth. Full mesh files and full URDF come from the upstream go2_nav2_ros2 repo. -->
 <robot name="go2" xmlns:xacro="http://www.ros.org/wiki/xacro">
   <!-- Include base GO2 description from upstream -->
   <!-- xacro:include filename="$(find go2_description)/xacro/go2_base.xacro"/ -->
-  <!-- ══════════════════════════════════════════════════════
-       RGB-D Camera — mounted on GO2 head
-       Add this block to your go2_robot.xacro
-       ══════════════════════════════════════════════════════ -->
+  <!-- RGB-D Camera — mounted on GO2 head -->
   <link name="camera_link">
     <visual>
@@ -55,6 +46,5 @@
     <origin xyz="0 0 0" rpy="-1.5708 0 -1.5708"/>
   </joint>
-  <!-- Depth camera sensor — requires LIBGL_DRI3_DISABLE=1 passed to gzserver
-       via SetEnvironmentVariable in gazebo_launch.py for OGRE to init correctly. -->
+  <!-- Depth camera sensor — requires LIBGL_DRI3_DISABLE=1 passed to gzserver via gazebo_launch.py for OGRE to init correctly. -->
   <gazebo reference="camera_link">
     <sensor type="depth" name="go2_camera">

File: go2_description/xacro/hokuyo_utm30lx.urdf.xacro (robot description, xacro)
@@ -73,42 +73,4 @@
       </gazebo>
     </xacro:macro>
-    <!-- <xacro:macro name="hokuyo_utm30lx_gpu" params="name parent *origin ros_topic update_rate ray_count min_angle max_angle">
-      <xacro:hokuyo_utm30lx_model name="${name}" parent="${parent}">
-        <xacro:insert_block name="origin" />
-      </xacro:hokuyo_utm30lx_model>
-      <gazebo reference="${name}_frame">
-        <sensor type="gpu_ray" name="${name}">
-          <update_rate>${update_rate}</update_rate>
-          <pose>0 0 0 0 0 0</pose>
-          <visualize>true</visualize>
-          <ray>
-            <scan>
-              <horizontal>
-                <samples>${ray_count}</samples>
-                <resolution>1</resolution>
-                <min_angle>${min_angle * M_PI/180}</min_angle>
-                <max_angle>${max_angle * M_PI/180}</max_angle>
-              </horizontal>
-            </scan>
-            <range>
-              <min>0.2</min>
-              <max>30.0</max>
-              <resolution>0.01</resolution>
-            </range>
-            <noise>
-              <type>gaussian</type>
-              <mean>0.0</mean>
-              <stddev>0.004</stddev>
-            </noise>
-          </ray>
-          <plugin name="gazebo_ros_${name}_controller" filename="libgazebo_ros_ray_sensor.so">
-            <ros>
-              <argument>~/out:=${ros_topic}</argument>
-            </ros>
-            <output_type>sensor_msgs/LaserScan</output_type>
-            <min_intensity>100.0</min_intensity>
-          </plugin>
-        </sensor>
-      </gazebo>
-    </xacro:macro> -->
+    <!-- GPU ray variant (unused): hokuyo_utm30lx_gpu macro omitted — use hokuyo_utm30lx with type="ray" above -->
 </robot>
